Commit message: added forward kinematics code

File: abb_irb120_support/urdf/irb120_3_58_macro.xacro (robot description, xacro)
@@ -217,5 +217,5 @@
     <link name="tool0" />
     <joint name="link_6-tool0" type="fixed">
-      <origin xyz="0 0 0" rpy="0 ${radians(90)} 0" />
+      <origin xyz="0 0 0" rpy="0 1.570796 0" />
       <parent link="flange" />
       <child link="tool0" />
